File: pcb/bakenko_65_iso.kicad_pcb (KiCad board)
At the start: 2 copper layers, 303.8 x 94.2 mm, 179 parts, among them J1 JST SH 4-pin, J2 Conn_01x02_MountingPin, K1 BUTTON-4P, Q1 AO3407A, U1 XC6206P302MR-G, U2 NRF52840 aQFN73, U3 MCP73831, X1 32MHz, X2 32.768KHz

Commit message: WIP + Cleaned repository
Parts:
- removed the C1 at (118.0, 49.4)
- removed the C11 at (114.8, 55.0)
- removed the C2 at (122.2, 46.5)
- removed the C20 at (127.5, 51.6)
- removed K1: BUTTON-4P, Seeed Studio XIAO nRF52840 v1.1:SW4-SMD-2.8-2.6X1.6X0.53MM
- removed R4, R5: 33R, Resistor_SMD:R_0402_1005Metric
- added C12: 100nF, Capacitor_SMD:C_0402_1005Metric, B.Cu at (136.1, 35.2)
- added C14: 1uF, Capacitor_SMD:C_0603_1608Metric, B.Cu at (137.7, 29.1)
- added C6: 4.7uF, Capacitor_SMD:C_0603_1608Metric, B.Cu at (146.6, 34.4)
- added C8: 100nF, Capacitor_SMD:C_0402_1005Metric, B.Cu at (142.8, 43.5)
- added REF**: STAB_MX_ISO-ROT, PCM_marbastlib-mx:STAB_MX_ISO-ROT, F.Cu at (367.3, 56.0)
- added REF**: STAB_MX_2u, PCM_marbastlib-mx:STAB_MX_2u, F.Cu at (360.1, 27.4)
- added REF**: STAB_MX_6.25u, PCM_marbastlib-mx:STAB_MX_6.25u, F.Cu at (224.4, 103.6)
- added SW1: SW_Omron_B3FS, Button_Switch_SMD:SW_SPST_TS-1088-xR020, F.Cu at (185.0, 104.8)
- C10: renamed from C12; moved to B.Cu
- C11: renamed from C23; value 100nF -> 100pF
- C13: renamed from C5; moved to B.Cu
- C15: renamed from C27; footprint Capacitor_SMD:C_0402_1005Metric -> Capacitor_SMD:C_0603_1608Metric; moved to B.Cu
- C20: renamed from C21; footprint Capacitor_SMD:C_0402_1005Metric -> Capacitor_SMD:C_0603_1608Metric
- C21: renamed from C25; footprint Capacitor_SMD:C_0402_1005Metric -> Capacitor_SMD:C_0603_1608Metric
- X1: footprint Crystal:Crystal_SMD_Abracon_ABM3C-4Pin_5.0x3.2mm -> Crystal:Crystal_SMD_2016-4Pin_2.0x1.6mm
- X2: footprint Crystal:Crystal_SMD_Abracon_ABS25-4Pin_8.0x3.8mm -> Crystal:Crystal_SMD_3215-2Pin_3.2x1.5mm
- moved C15 140.5 mm to (137.7, 32.4), turned to -45 degrees
- moved ANT1 95.0 mm to (131.5, 21.2), turned to 90 degrees
- moved L2 87.4 mm to (131.5, 24.8), turned to 90 degrees
- moved L3 83.1 mm to (130.1, 25.9), turned to 180 degrees
- moved C33 80.6 mm to (131.5, 27.1), turned to 90 degrees
- moved C13 54.5 mm to (135.8, 33.4), turned to 180 degrees
- moved C10 51.0 mm to (133.0, 37.7), turned to 90 degrees
- moved C2 43.1 mm to (136.5, 30.0)
- moved X1 40.6 mm to (134.5, 31.5)
- moved C1 38.9 mm to (132.5, 31.6)
- moved C7 32.5 mm to (144.8, 41.8), turned to 135 degrees
- moved L1 28.3 mm to (131.6, 35.9), turned to 90 degrees
- moved C4 28.3 mm to (131.0, 34.4), turned to 0 degrees
- moved C3 27.8 mm to (133.0, 36.3), turned to 180 degrees
- moved C20 25.8 mm to (147.7, 35.5), turned to -135 degrees
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- renumbered C6 to C1, C9 to C17, C16 to C18, C8 to C2, C17 to C3, C3 to C30, C4 to C31, C14 to C33, C19 to C4, C10 to C5, C13 to L1, C15 to L2, C18 to L3
Connections:
- net Net-(U2-P0.01) renamed /X2_N
- C1 pad 1: Net-(C6-Pad1) -> /XC_N
- C17 pad 2: Net-(U2-P0.00) -> /X2_P
- C2 pad 1: Net-(C8-Pad1) -> GND
- C2 pad 2: GND -> /XC_P
- C3 pad 1: Net-(C17-Pad1) -> GND
- C30 pad 2: /3V3 -> +3V3
- C31 pad 1: /VIN -> VIN
- C4 pad 1: Net-(C17-Pad1) -> GND
- C7 pad 1: /3V3 -> GND
- C7 pad 2: GND -> +3V3
- D1 pad 1: /VIN -> VIN
- Q1 pad 2: VBUS -> VIN
- Q1 pad 3: /VIN -> VBUS
- R1 pad 1: GND -> VBUS
- R1 pad 2: VBUS -> GND
- R10 pad 1: /3V3 -> /RESET
- R10 pad 2: /RESET -> +3V3
- R12 pad 2: Net-(U3-V_{SS}) -> GND
- U1 pad 2: /3V3 -> +3V3
- U1 pad 3: /VIN -> VIN
- U2 pad A10: unconnected-(U2-P0.29-PadA10) -> COL4
- U2 pad A12: unconnected-(U2-P0.02-PadA12) -> COL3
- U2 pad A14: unconnected-(U2-P1.15-PadA14) -> COL2
- U2 pad A16: unconnected-(U2-P1.13-PadA16) -> COL1
- U2 pad A20: unconnected-(U2-P1.10-PadA20) -> COL0
- U2 pad A23: unconnected-(U2-XC2-PadA23) -> /XC_P
- U2 pad AC9: /P0.14_~{READ_BAT} -> unconnected-(U2-P0.14-PadAC9)
- U2 pad AD10: unconnected-(U2-P0.15-PadAD10) -> /P0.14_~{READ_BAT}
- U2 pad AD12: unconnected-(U2-P0.17-PadAD12) -> /RESET
- U2 pad AD4: Net-(U2-D-) -> /USB_D-
- U2 pad AD6: Net-(U2-D+) -> /USB_D+
- U2 pad B19: /P1.11_TX_D6 -> unconnected-(U2-P1.11-PadB19)
- U2 pad B24: unconnected-(U2-XC1-PadB24) -> /XC_N
- U2 pad B3: Net-(U2-DCC) -> GND
- U2 pad D2: Net-(U2-P0.00) -> /X2_P
- U2 pad H2: COL0 -> unconnected-(U2-P0.27-PadH2)
- U2 pad J24: ROW4 -> ROW0
- U2 pad K2: COL1 -> unconnected-(U2-P0.05-PadK2)
- U2 pad L24: ROW3 -> ROW1
- U2 pad M2: COL4 -> unconnected-(U2-P0.07-PadM2)
- U2 pad P2: COL3 -> unconnected-(U2-P1.08-PadP2)
- U2 pad T2: COL2 -> unconnected-(U2-P0.11-PadT2)
- U2 pad U24: ROW0 -> ROW3
- U2 pad W24: ROW1 -> ROW4
- U3 pad 2: Net-(U3-V_{SS}) -> GND
- X1 pad 1: Net-(C8-Pad1) -> /XC_P
- X1 pad 2: GND -> /XC_N
- X1 pad 3: Net-(C6-Pad1) -> (no net)
- X1 pad 4: GND -> (no net)
- X2 pad 2: GND -> /X2_P
Routing:
- net ROW4: track 335.5 -> 72.5 mm
- net ROW2: track 282.6 -> 28.5 mm
- net COL12: track 334.0 -> 86.1 mm
- net ROW3: track 290.0 -> 48.0 mm
- net COL11: track 313.1 -> 87.0 mm
- net COL14: track 271.7 -> 76.2 mm
- net ROW0: track 303.4 -> 117.0 mm, vias 2 -> 0
- net COL13: track 249.6 -> 80.3 mm
- net /3V3: track 134.1 -> 0.00 mm, vias 7 -> 0
- net COL10: track 185.8 -> 67.0 mm
- net /RESET: track 92.0 -> 0.60 mm, vias 2 -> 0
- net COL0: track 125.6 -> 40.1 mm, vias 2 -> 1
- net COL8: track 148.1 -> 67.0 mm
- net ROW1: track 360.1 -> 281.1 mm
- net COL9: track 167.0 -> 93.0 mm
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Other:
- board text added: "Bakeneko65-ISO v4.0"
- board text removed: "Bakeneko65 v3.0"

Commit message: 🧹Cleaned more up and updated the readme
Parts:
- added D47: 1N4148, Diode_SMD:D_SOD-123, B.Cu at (118.4, 85.3)
- added G***: LOGO, LOGO, F.Cu at (255.1, 102.5)
- added MX46: 1u, PCM_marbastlib-mx:SW_MX_1u, F.Cu at (126.8, 84.5)
- MX1, MX10, MX11, MX12, MX13, MX15, MX17, MX18, MX19, MX2, MX20, MX21, MX22, MX23, MX24, MX25, MX26, MX27, MX28, MX3, MX30, MX32, MX33, MX34, MX35, MX36, MX37, MX38, MX39, MX4, MX40, MX41, MX42, MX43, MX44, MX5, MX6, MX7, MX8, MX9: footprint MX_Only:MXOnly-1U-NoLED -> PCM_marbastlib-mx:SW_MX_1u
- MX14: footprint MX_Only:MXOnly-2U-NoLED -> PCM_marbastlib-mx:SW_MX_1u
- MX16: footprint MX_Only:MXOnly-1.5U-NoLED -> PCM_marbastlib-mx:SW_MX_1.5u
- MX29: footprint MX_Only:MXOnly-ISO-ROTATED-ReversedStabilizers-NoLED -> PCM_marbastlib-mx:SW_MX_1u
- MX31: footprint MX_Only:MXOnly-1.75U-NoLED -> PCM_marbastlib-mx:SW_MX_1.75u
- MX45: footprint MX_Only:MXOnly-2.25U-NoLED -> PCM_marbastlib-mx:SW_MX_1.25u
- MX47: renamed from MX46; footprint MX_Only:MXOnly-1U-NoLED -> PCM_marbastlib-mx:SW_MX_1u
- MX48: renamed from MX47; footprint MX_Only:MXOnly-1U-NoLED -> PCM_marbastlib-mx:SW_MX_1u
- MX49: renamed from MX48; footprint MX_Only:MXOnly-1U-NoLED -> PCM_marbastlib-mx:SW_MX_1u
- MX50: renamed from MX49; footprint MX_Only:MXOnly-1U-NoLED -> PCM_marbastlib-mx:SW_MX_1u
- MX51: renamed from MX50; footprint MX_Only:MXOnly-1U-NoLED -> PCM_marbastlib-mx:SW_MX_1u
- MX52: renamed from MX51; footprint MX_Only:MXOnly-1U-NoLED -> PCM_marbastlib-mx:SW_MX_1u
- MX53: renamed from MX52; footprint MX_Only:MXOnly-1U-NoLED -> PCM_marbastlib-mx:SW_MX_1u
- MX54: renamed from MX53; footprint MX_Only:MXOnly-1U-NoLED -> PCM_marbastlib-mx:SW_MX_1u
- MX55: renamed from MX54; footprint MX_Only:MXOnly-1U-NoLED -> PCM_marbastlib-mx:SW_MX_1u
- MX56: renamed from MX55; footprint MX_Only:MXOnly-1U-NoLED -> PCM_marbastlib-mx:SW_MX_1u
- MX57: renamed from MX56; footprint MX_Only:MXOnly-1.75U-NoLED -> PCM_marbastlib-mx:SW_MX_1.75u
- MX58: renamed from MX57; footprint MX_Only:MXOnly-1U-NoLED -> PCM_marbastlib-mx:SW_MX_1u
- MX59: renamed from MX58; footprint MX_Only:MXOnly-1U-NoLED -> PCM_marbastlib-mx:SW_MX_1u
- MX60: renamed from MX59; footprint MX_Only:MXOnly-1.25U-NoLED -> PCM_marbastlib-mx:SW_MX_1.25u
- MX61: renamed from MX60; footprint MX_Only:MXOnly-1.25U-NoLED -> PCM_marbastlib-mx:SW_MX_1.25u
- MX62: renamed from MX61; footprint MX_Only:MXOnly-1.25U-NoLED -> PCM_marbastlib-mx:SW_MX_1.25u
- MX63: renamed from MX62; footprint MX_Only:MXOnly-6.25U-ReversedStabilizers-NoLED -> PCM_marbastlib-mx:SW_MX_1u
- MX64: renamed from MX63; footprint MX_Only:MXOnly-1.25U-NoLED -> PCM_marbastlib-mx:SW_MX_1.25u
- MX65: renamed from MX64; footprint MX_Only:MXOnly-1.25U-NoLED -> PCM_marbastlib-mx:SW_MX_1.25u
- MX66: renamed from MX65; footprint MX_Only:MXOnly-1U-NoLED -> PCM_marbastlib-mx:SW_MX_1u
- MX67: renamed from MX66; footprint MX_Only:MXOnly-1U-NoLED -> PCM_marbastlib-mx:SW_MX_1u
- MX68: renamed from MX67; footprint MX_Only:MXOnly-1U-NoLED -> PCM_marbastlib-mx:SW_MX_1u
- moved SW1 11.1 mm to (195.8, 102.4)
- moved MX45 9.53 mm to (105.3, 84.5)
- moved D46 7.94 mm to (114.8, 85.3)
- moved C3 4.90 mm to (128.1, 36.4), turned to 0 degrees
- moved X1 3.83 mm to (133.5, 35.2), turned to -90 degrees
- moved C2 3.66 mm to (134.1, 32.7)
- moved C1 3.32 mm to (131.7, 34.9)
- moved C17 2.66 mm to (143.6, 29.4), turned to -135 degrees
- moved C18 2.25 mm to (145.4, 31.2), turned to -135 degrees
- moved L1 2.05 mm to (129.6, 35.9)
- moved L3 2.05 mm to (128.1, 25.9)
- moved ANT1 2.05 mm to (129.5, 21.2)
- moved C33 2.05 mm to (129.5, 27.1)
- moved C4 2.05 mm to (129.0, 34.4)
- moved L2 2.05 mm to (129.5, 24.8)
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- renumbered D47 to D48, D48 to D49, D49 to D50, D50 to D51, D51 to D52, D52 to D53, D53 to D54, D54 to D55, D55 to D56, D56 to D57, D57 to D58, D58 to D59, D59 to D60, D60 to D61, D61 to D62, D62 to D63, D63 to D64, D64 to D65, D65 to D66, D66 to D67, D67 to D68, D68 to D69
Connections:
- U2 pad B3: GND -> unconnected-(U2-DCC-PadB3)
- U2 pad G1: COL5 -> COL10
- U2 pad J1: COL6 -> COL9
- U2 pad L1: COL7 -> COL8
- U2 pad N1: COL8 -> COL7
- U2 pad R1: COL9 -> COL6
- U2 pad U1: COL10 -> COL5
- X1 pad 2: /XC_N -> GND
- X1 pad 3: (no net) -> /XC_N
- X1 pad 4: (no net) -> GND
Routing:
- net ROW4: track 72.5 -> 357.0 mm
- net COL14: track 76.2 -> 344.4 mm, vias 0 -> 2
- net ROW3: track 48.0 -> 314.5 mm
- net ROW2: track 28.5 -> 292.8 mm
- net COL13: track 80.3 -> 328.0 mm, vias 0 -> 2
- net COL12: track 86.1 -> 310.7 mm, vias 0 -> 2
- net ROW0: track 117.0 -> 328.4 mm
- net COL11: track 87.0 -> 293.0 mm, vias 0 -> 2
- net COL10: track 67.0 -> 231.0 mm, vias 0 -> 1
- net COL9: track 93.0 -> 237.6 mm, vias 0 -> 1
- net COL8: track 67.0 -> 192.0 mm, vias 0 -> 1
- net COL7: track 67.0 -> 171.2 mm, vias 0 -> 1
- net COL0: track 40.1 -> 128.6 mm
- net COL6: track 87.0 -> 171.6 mm, vias 0 -> 1
- net COL5: track 67.0 -> 132.0 mm, vias 0 -> 1
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Other:
- board text added: "RESET"

Commit message: Cleaning zones and moving antenna
Parts:
- moved ANT1 37.4 mm to (96.9, 39.5), turned to 180 degrees
- moved L2 32.5 mm to (100.5, 39.5), turned to 180 degrees
- moved L3 30.5 mm to (101.6, 40.9), turned to -90 degrees
- moved C33 29.5 mm to (102.8, 39.5), turned to 180 degrees
- moved R10 21.4 mm to (186.1, 103.5)
- moved C26 19.0 mm to (186.1, 101.1)
- moved C3 5.92 mm to (131.8, 41.1), turned to 90 degrees
- moved C4 4.78 mm to (129.8, 39.1), turned to -90 degrees
- moved L1 4.10 mm to (131.3, 39.6), turned to 180 degrees
- turned SW1 to 0 degrees
Routing:
- net Net-(C33-Pad1): track 8.04 -> 35.7 mm
- net Net-(U2-ANT): track 13.2 -> 7.89 mm
- net GND: track 34.3 -> 35.0 mm, vias 97 -> 113
- net ROW0: track 328.4 -> 327.7 mm, vias 0 -> 2
- net Net-(C33-Pad2): vias 1 -> 0
- net COL0: vias 1 -> 2
- net /P0.31_AIN7_BAT: vias 3 -> 2

Commit message: Connecting reset and reducing errors and warnings
Parts:
- moved R12 0.84 mm to (151.4, 32.4)
Connections:
- U2 pad A10: COL4 -> COL2
- U2 pad A14: COL2 -> COL4
- U2 pad A8: /P0.31_AIN7_BAT -> unconnected-(U2-P0.31-PadA8)
- U2 pad AD10: /P0.14_~{READ_BAT} -> /P0.31_AIN7_BAT
- U2 pad AD8: unconnected-(U2-P0.13-PadAD8) -> /P0.14_~{READ_BAT}
Routing:
- net /RESET: track 0.60 -> 98.3 mm, vias 0 -> 2
- net +3V3: track 51.3 -> 140.7 mm, vias 5 -> 7
- net GND: track 35.0 -> 98.2 mm, vias 113 -> 109
- net COL2: track 82.7 -> 130.9 mm, vias 1 -> 3
- net Net-(D2-A): track 0.00 -> 12.4 mm
- net VBUS: track 20.2 -> 28.4 mm
- net Net-(C33-Pad1): track 35.7 -> 28.0 mm
- net /P0.31_AIN7_BAT: track 5.04 -> 12.6 mm, vias 2 -> 0
- net Net-(D56-A): track 0.00 -> 6.41 mm
- net Net-(D52-A): track 0.00 -> 6.41 mm
- net Net-(D8-A): track 0.00 -> 6.41 mm
- net Net-(D38-A): track 0.00 -> 6.41 mm
- net Net-(D37-A): track 0.00 -> 6.41 mm
- net Net-(D36-A): track 0.00 -> 6.41 mm
- net Net-(D21-A): track 0.00 -> 4.82 mm
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
Commit message: Adding changes thanks to comment from devzone nordic
Parts:
- J1: footprint Connector_JST:JST_SH_SM04B-SRSS-TB_1x04-1MP_P1.00mm_Horizontal -> Connector_Molex:Molex_Pico-EZmate_78171-0004_1x04-1MP_P1.20mm_Vertical
- moved C3 4.27 mm to (135.8, 39.7), turned to -45 degrees
- moved C4 2.70 mm to (132.5, 39.2)
- moved L1 2.69 mm to (133.9, 39.7)
- moved C10 0.52 mm to (132.5, 37.7), turned to 180 degrees
Connections:
- C3 pad 1: GND -> Net-(U2-VSS_PA)
- J1 pad MP: (no net) -> GND
- U2 pad F23: GND -> Net-(U2-VSS_PA)
Routing:
- net COL0: track 128.6 -> 274.8 mm, vias 1 -> 4
- net COL1: track 99.2 -> 207.2 mm, vias 2 -> 6
- net GND: track 98.2 -> 103.1 mm, vias 109 -> 119
- net ROW0: track 328.5 -> 333.2 mm, vias 2 -> 0
- net Net-(U2-ANT): track 7.89 -> 4.47 mm
- net Net-(U2-VSS_PA): track 0.00 -> 2.87 mm
- net Net-(C33-Pad1): track 28.0 -> 30.4 mm
- net +3V3: track 140.7 -> 139.2 mm

Commit message: Final changes before pcb-assebly
Parts:
- J1: value JST SH 4-pin -> Molex_Pico-EZmate_781710004
Changed lines of the file:
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@@
 			)
 		)
-		(property "Value" "JST SH 4-pin"
+		(property "Value" "Molex_Pico-EZmate_781710004"
 			(at 0 -3.72 90)
 			(layer "B.Fab")
@@
 		(descr "SMD2016/4, Crystal, 2.0x1.6mm package, SMD, generated with kicad-footprint-generator make_crystal.py, http://www.q-crystal.com/upload/5/2015552223166229.pdf")
 		(property "Reference" "X1"
-			(at 1.25 2 180)
+			(at 1.25 2 0)
 			(layer "B.SilkS")
 			(effects
@@
 	)
 	(segment
+		(start 137.937556 38.560139)
+		(end 137.942424 38.560139)
+		(width 0.15)
+		(layer "B.Cu")
+		(net "Net-(U2-VSS_PA)")
+	)
+	(segment
+		(start 137.937556 38.736915)
+		(end 137.322892 39.351579)
+		(width 0.15)
+		(layer "B.Cu")
+		(net "Net-(U2-VSS_PA)")
+	)
+	(segment
+		(start 137.322892 39.351579)
+		(end 135.503349 39.351579)
+		(width 0.15)
+		(layer "B.Cu")
+		(net "Net-(U2-VSS_PA)")
+	)
+	(segment
+		(start 137.937556 38.560139)
+		(end 137.937556 38.736915)
+		(width 0.15)
+		(layer "B.Cu")
+		(net "Net-(U2-VSS_PA)")
+	)
+	(segment
 		(start 134.09276 34.955118)
 		(end 134.66776 35.530118)
@@
 		(net "Net-(U3-PROG)")
 	)
-	(segment
-		(start 137.937556 38.560139)
-		(end 137.942424 38.560139)
-		(width 0.15)
-		(layer "B.Cu")
-		(net "Net-(U2-VSS_PA)")
-	)
-	(segment
-		(start 137.937556 38.736915)
-		(end 137.322892 39.351579)
-		(width 0.15)
-		(layer "B.Cu")
-		(net "Net-(U2-VSS_PA)")
-	)
-	(segment
-		(start 137.322892 39.351579)
-		(end 135.503349 39.351579)
-		(width 0.15)
-		(layer "B.Cu")
-		(net "Net-(U2-VSS_PA)")
-	)
-	(segment
-		(start 137.937556 38.560139)
-		(end 137.937556 38.736915)
-		(width 0.15)
-		(layer "B.Cu")
-		(net "Net-(U2-VSS_PA)")
-	)
 	(zone
